File: LinePCB.kicad_pcb (KiCad board)
At the start: 4 copper layers, 178 x 169.8 mm, 225 parts, among them J1 Conn_01x12, J3 Conn_01x03, J4 Conn_01x05_Pin, U1 MCP3008, U10 Optocoupler, U11 210, U12 2200, U13 2200, U14 210, U15 Oprocoupler, U16 10k, U17 N channel, U18 D, U19 10K, U2 MCP3008, U20 Conn_01x02, U21 V_Regulator3.3v, U22 V_Regulator5v, U3 MCP3008, U4 MCP3008, U5 MCP3008, U6 MCP3008, U7 30k, U8 115k, U9 BSP89

Commit message: Fixed Routing Errors
Parts:
- removed J3: Conn_01x03, Connector_JST:JST_XH_B3B-XH-A_1x03_P2.50mm_Vertical
- moved U22 6.86 mm to (115.0, 45.3), turned to -56 degrees
- moved U21 4.57 mm to (70.4, 35.3), turned to -124 degrees
- moved J4 3.30 mm to (65.5, 36.3), turned to -124 degrees
Routing:
- net 12V: track 345.8 -> 225.9 mm, vias 4 -> 1
- net 48V: track 312.7 -> 193.1 mm, vias 5 -> 3
- net 3.3V: track 1010.7 -> 985.1 mm, vias 56 -> 53
- net 5V: track 54.2 -> 69.4 mm
- net GND: track 1145.7 -> 1138.2 mm
- net Ch33: track 138.9 -> 139.7 mm
Other:
- outline, holes or cut-outs redrawn

Commit message: Fixed Floating Ground
Routing:
- net GND: track 1138.2 -> 1098.2 mm
Changed lines of the file:
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@@
-	)
-	(segment
-		(start 41.0743 100.2557)
-		(end 39.73 101.6)
-		(width 0.2)
-		(layer "In1.Cu")
-		(net 5)
 	)
 	(segment
@@
 	)
 	(segment
-		(start 41.0743 91.288)
-		(end 41.0743 100.2557)
-		(width 0.2)
-		(layer "In1.Cu")
-		(net 5)
-	)
-	(segment
 		(start 142.921757 174.55)
 		(end 144.75 174.55)
@@
 	)
 	(segment
-		(start 42.226 91.288)
-		(end 41.0743 91.288)
-		(width 0.2)
-		(layer "In1.Cu")
-		(net 5)
-	)
-	(segment
 		(start 53.2 37.9)
 		(end 52.7123 38.3877)
@@
 	)
 	(segment
-		(start 42.226 91.288)
-		(end 41.0743 91.288)
-		(width 0.2)
-		(layer "In2.Cu")
-		(net 5)
-	)
-	(segment
-		(start 41.0743 91.7199)
-		(end 37.8202 94.974)
-		(width 0.2)
-		(layer "In2.Cu")
-		(net 5)
-	)
-	(segment
 		(start 31.2406 104.0275)
 		(end 37.3025 104.0275)
@@
 	)
 	(segment
-		(start 37.8202 94.974)
-		(end 16.0232 94.974)
-		(width 0.2)
-		(layer "In2.Cu")
-		(net 5)
-	)
-	(segment
 		(start 25.491697 122.407384)
 		(end 25.491697 123.54017)
@@
 		(width 0.2)
 		(layer "In2.Cu")
-		(net 5)
-	)
-	(segment
-		(start 41.0743 91.288)
-		(end 41.0743 91.7199)
-		(width 0.2)
-		(layer "In2.Cu")
